File: main_board_v1/audio.kicad_sch (KiCad schematic)
At the start: 30 parts, among them J10 PJ-342, U10 TLV320DAC3101IRHBR, U9 LD1117S18TR_SOT223

Commit message: cosmetic change
Other:
- note removed: "oops"
Changed lines of the file:
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@@
-    (effects (font (size 1.27 1.27)) (justify left bottom))
-  )
-  (text "oops" (at 153.035 105.41 0)
     (effects (font (size 1.27 1.27)) (justify left bottom))
   )
